Commit message: Made the robot more robust

File: turtlebot3_burger_gripper.urdf.xacro (robot description, xacro)
@@ -212,15 +212,15 @@
     <parent link="gripper_beam"/>
     <child link="gripper_left"/>
-    <origin xyz="0.07 0.0 0.03" rpy="0 0 0"/>
+    <origin xyz="0.08 0.0 0.03" rpy="0 0 0"/>
   </joint>
   <link name="gripper_left" type="fixed">
     <visual>
       <geometry>
-        <box size="0.01 0.01 0.06"/>
-      </geometry>
-    </visual>
-    <collision>
-      <geometry>
-        <box size="0.01 0.01 0.06"/>
+        <box size="0.01 0.01 0.08"/>
+      </geometry>
+    </visual>
+    <collision>
+      <geometry>
+        <box size="0.01 0.01 0.08"/>
       </geometry>
     </collision>
@@ -229,15 +229,15 @@
     <parent link="gripper_beam"/>
     <child link="gripper_right"/>
-    <origin xyz="-0.07 0.0 0.03" rpy="0 0 0"/>
+    <origin xyz="-0.08 0.0 0.03" rpy="0 0 0"/>
   </joint>
   <link name="gripper_right" type="fixed">
     <visual>
       <geometry>
-        <box size="0.01 0.01 0.06"/>
-      </geometry>
-    </visual>
-    <collision>
-      <geometry>
-        <box size="0.01 0.01 0.06"/>
+        <box size="0.01 0.01 0.08"/>
+      </geometry>
+    </visual>
+    <collision>
+      <geometry>
+        <box size="0.01 0.01 0.08"/>
       </geometry>
     </collision>
