Commit message: Changed turtlebot models
Scout is now white.
Grippers gripper is now red.
Model collision is raised so a robot is of the same size on both scans.
Grippers bottom scan is changed so it only scans between -45 and 45 degrees this breaks the multi_agent_cluster package.

File: turtlebot3_burger_gripper.gazebo.xacro (robot description, xacro)
@@ -36,14 +36,14 @@
   </gazebo>
   <gazebo reference="gripper_base_joint">
-    <material>Gazebo/DarkGrey</material>
+    <material>Gazebo/Red</material>
   </gazebo>
   <gazebo reference="gripper_beam">
-    <material>Gazebo/DarkGrey</material>
+    <material>Gazebo/Red</material>
   </gazebo>
   <gazebo reference="gripper_left">
-    <material>Gazebo/DarkGrey</material>
+    <material>Gazebo/Red</material>
   </gazebo>
   <gazebo reference="gripper_right">
-    <material>Gazebo/DarkGrey</material>
+    <material>Gazebo/Red</material>
   </gazebo>
   <gazebo reference="imu_link">
@@ -145,13 +145,13 @@
         <scan>
           <horizontal>
-            <samples>360</samples>
+            <samples>90</samples>
             <resolution>1</resolution>
-            <min_angle>0.0</min_angle>
-            <max_angle>6.28319</max_angle>
+            <min_angle>-0.7854</min_angle>
+            <max_angle>0.7854</max_angle>
           </horizontal>
         </scan>
         <range>
-          <min>0.120</min>
-          <max>3.5</max>
+          <min>0.1</min>
+          <max>2.0</max>
           <resolution>0.015</resolution>
         </range>

File: turtlebot3_burger_gripper.urdf.xacro (robot description, xacro)
@@ -19,7 +19,7 @@
     </visual>
     <collision>
-      <origin xyz="-0.032 0 0.070" rpy="0 0 0"/>
-      <geometry>
-        <box size="0.140 0.140 0.143"/>
+      <origin xyz="-0.032 0 0.100" rpy="0 0 0"/>
+      <geometry>
+        <box size="0.140 0.140 0.203"/>
       </geometry>
     </collision>

File: turtlebot3_burger_scout.gazebo.xacro (robot description, xacro)
@@ -4,5 +4,5 @@
   <xacro:arg name="imu_visual"   default="false"/>
   <gazebo reference="base_link">
-    <material>Gazebo/DarkGrey</material>
+    <material>Gazebo/White</material>
   </gazebo>
   <gazebo reference="wheel_left_link">

File: turtlebot3_burger_scout.urdf.xacro (robot description, xacro)
@@ -2,5 +2,5 @@
 <robot name="turtlebot3_burger_gripper" xmlns:xacro="http://ros.org/wiki/xacro">
   <xacro:include filename="$(find turtlebot3_description)/urdf/common_properties.xacro"/>
-  <xacro:include filename="$(find turtlebot3_description)/urdf/turtlebot3_burger_gripper.gazebo.xacro"/>
+  <xacro:include filename="$(find turtlebot3_description)/urdf/turtlebot3_burger_scout.gazebo.xacro"/>
   <!-- Robot Base -->
   <link name="base_footprint"/>
@@ -19,7 +19,7 @@
     </visual>
     <collision>
-      <origin xyz="-0.032 0 0.070" rpy="0 0 0"/>
+      <origin xyz="-0.032 0 0.100" rpy="0 0 0"/>
       <geometry>
-        <box size="0.140 0.140 0.143"/>
+        <box size="0.140 0.140 0.203"/>
       </geometry>
     </collision>
